File: breakout board/breakout board.kicad_pcb (KiCad board)
At the start: 4 copper layers, 30.6 x 63.3 mm, 28 parts, among them J1 USB_B_Micro, J2 Conn_01x18, J3 Screw_Terminal_01x02, J4 Conn_01x18, SW1 SW_SPDT, U1 AMS1117-3.3, U2 STM32F302C8Tx, Y1 X322516MLB4SI

Commit message: Add files via upload
Routing:
- net +3V3: track 59.1 -> 147.7 mm, vias 6 -> 9
- net VBUS: track 54.0 -> 55.7 mm
Other:
- board size 30.6 x 63.3 mm -> 28 x 63.3 mm
Changed lines of the file:
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@@
     )
   )
-  (gr_line (start 80.57868 86.971573) (end 80.57868 29.7) (layer "Edge.Cuts") (width 0.05))
-  (gr_arc (start 50.02132 29.7) (mid 50.9 27.57868) (end 53.02132 26.7) (layer "Edge.Cuts") (width 0.05))
-  (gr_arc (start 80.57868 86.971573) (mid 79.7 89.092893) (end 77.57868 89.971573) (layer "Edge.Cuts") (width 0.05))
-  (gr_line (start 53.05 89.971573) (end 77.57868 89.971573) (layer "Edge.Cuts") (width 0.05))
-  (gr_arc (start 77.57868 26.7) (mid 79.7 27.57868) (end 80.57868 29.7) (layer "Edge.Cuts") (width 0.05))
-  (gr_line (start 77.57868 26.7) (end 53.02132 26.7) (layer "Edge.Cuts") (width 0.05))
-  (gr_line (start 50.05 86.971573) (end 50.02132 29.7) (layer "Edge.Cuts") (width 0.05))
-  (gr_arc (start 53.05 89.971573) (mid 50.92868 89.092893) (end 50.05 86.971573) (layer "Edge.Cuts") (width 0.05))
+  (gr_line (start 79.525 86.960787) (end 79.525 29.689214) (layer "Edge.Cuts") (width 0.05))
+  (gr_line (start 76.525 26.7) (end 54.51764 26.7) (layer "Edge.Cuts") (width 0.05))
+  (gr_line (start 54.54632 89.971573) (end 76.525 89.960787) (layer "Edge.Cuts") (width 0.05))
+  (gr_arc (start 51.51764 29.7) (mid 52.39632 27.57868) (end 54.51764 26.7) (layer "Edge.Cuts") (width 0.05))
+  (gr_arc (start 79.525 86.960787) (mid 78.64632 89.082107) (end 76.525 89.960787) (layer "Edge.Cuts") (width 0.05))
+  (gr_arc (start 76.525 26.7) (mid 78.64632 27.57868) (end 79.525 29.7) (layer "Edge.Cuts") (width 0.05))
+  (gr_line (start 51.54632 86.971573) (end 51.51764 29.7) (layer "Edge.Cuts") (width 0.05))
+  (gr_arc (start 54.54632 89.971573) (mid 52.425 89.092893) (end 51.54632 86.971573) (layer "Edge.Cuts") (width 0.05))
+  (dimension (type aligned) (layer "Edge.Cuts")
+    (pts (xy 76.525 26.7) (xy 76.525 89.960787))
+    (height -4.45)
+    (gr_text "63.2608 mm" (at 79.825 58.330393 90) (layer "Edge.Cuts")
+      (effects (font (size 1 1) (thickness 0.15)))
+    )
+    (format (units 3) (units_format 1) (precision 4))
+    (style (thickness 0.1) (arrow_length 1.27) (text_position_mode 0) (extension_height 0.58642) (extension_offset 0.5) keep_text_aligned)
+  )
+  (dimension (type aligned) (layer "Edge.Cuts")
+    (pts (xy 51.51764 29.675) (xy 79.525 29.675))
+    (height -4.875)
+    (gr_text "28.0074 mm" (at 65.52132 23.65) (layer "Edge.Cuts")
+      (effects (font (size 1 1) (thickness 0.15)))
+    )
+    (format (units 3) (units_format 1) (precision 4))
+    (style (thickness 0.1) (arrow_length 1.27) (text_position_mode 0) (extension_height 0.58642) (extension_offset 0.5) keep_text_aligned)
+  )
   (segment (start 70.639411 50.792143) (end 70.639411 49.760589) (width 0.5) (layer "F.Cu") (net 1))
   (segment (start 72.221178 64.8) (end 73.4 64.8) (width 0.5) (layer "F.Cu") (net 1))
@@
   (segment (start 57.55 64.325) (end 58.203822 64.325) (width 0.3) (layer "F.Cu") (net 3))
   (segment (start 65.4 54.9) (end 66.775 54.9) (width 0.5) (layer "F.Cu") (net 3))
-  (segment (start 72.589411 63.810589) (end 72.22761 63.448788) (width 0.3) (layer "F.Cu") (net 3))
   (segment (start 70.337876 61.450532) (end 70.337876 61.451212) (width 0.3) (layer "F.Cu") (net 3))
+  (segment (start 72.22761 63.448788) (end 70.337876 63.448788) (width 0.3) (layer "F.Cu") (net 3))
   (segment (start 58.203822 64.325) (end 59.689411 62.839411) (width 0.3) (layer "F.Cu") (net 3))
   (segment (start 68.72 56.9) (end 68.72 56.845) (width 0.3) (layer "F.Cu") (net 3))
@@
   (segment (start 64.78 69.35) (end 64.78 67.666664) (width 0.3) (layer "F.Cu") (net 3))
   (segment (start 60.562124 61.966698) (end 59.689411 62.839411) (width 0.3) (layer "F.Cu") (net 3))
+  (segment (start 72.060589 60.689411) (end 72.064411 60.689411) (width 0.3) (layer "F.Cu") (net 3))
+  (segment (start 64.78 69.35) (end 65.7 69.35) (width 0.3) (layer "F.Cu") (net 3))
   (segment (start 72.060589 60.689411) (end 71.098997 60.689411) (width 0.3) (layer "F.Cu") (net 3))
   (segment (start 62.05 43.8) (end 62 43.75) (width 0.5) (layer "F.Cu") (net 3))
   (segment (start 64.65 41.1) (end 62 43.75) (width 0.3) (layer "F.Cu") (net 3))
-  (segment (start 72.22761 63.448788) (end 70.337876 63.448788) (width 0.3) (layer "F.Cu") (net 3))
+  (segment (start 72.064411 60.689411) (end 72.75 61.375) (width 0.3) (layer "F.Cu") (net 3))
   (segment (start 66.675 41.1) (end 64.65 41.1) (width 0.3) (layer "F.Cu") (net 3))
+  (segment (start 65.7 69.35) (end 65.725 69.325) (width 0.3) (layer "F.Cu") (net 3))
   (segment (start 71.098997 60.689411) (end 70.337876 61.450532) (width 0.3) (layer "F.Cu") (net 3))
+  (segment (start 72.589411 63.810589) (end 73.275 63.125) (width 0.3) (layer "F.Cu") (net 3))
+  (segment (start 72.589411 63.810589) (end 72.22761 63.448788) (width 0.3) (layer "F.Cu") (net 3))
   (segment (start 75 86.25) (end 77.43 86.25) (width 0.5) (layer "F.Cu") (net 3))
   (segment (start 77.43 86.25) (end 77.475 86.205) (width 0.5) (layer "F.Cu") (net 3))
@@
   (via (at 63.4 76.5) (size 0.8) (drill 0.4) (layers "F.Cu" "B.Cu") (free) (net 3))
   (via (at 56.65 65.7) (size 0.8) (drill 0.4) (layers "F.Cu" "B.Cu") (free) (net 3))
+  (via (at 72.75 61.375) (size 0.8) (drill 0.4) (layers "F.Cu" "B.Cu") (free) (net 3))
+  (via (at 65.725 69.325) (size 0.8) (drill 0.4) (layers "F.Cu" "B.Cu") (free) (net 3))
+  (via (at 73.275 63.125) (size 0.8) (drill 0.4) (layers "F.Cu" "B.Cu") (free) (net 3))
   (via (at 65.4 54.9) (size 0.8) (drill 0.4) (layers "F.Cu" "B.Cu") (free) (net 3))
   (via (at 62.05 45.9) (size 0.8) (drill 0.4) (layers "F.Cu" "B.Cu") (free) (net 3))
-  (segment (start 63.95 46.05) (end 64.15 46.25) (width 0.5) (layer "In1.Cu") (net 3))
+  (segment (start 58.7 63.65) (end 56.65 65.7) (width 0.3) (layer "In1.Cu") (net 3))
+  (segment (start 73.275 63.125) (end 74.349511 62.050489) (width 0.3) (layer "In1.Cu") (net 3))
+  (segment (start 65.725 69.325) (end 64.900489 68.500489) (width 0.3) (layer "In1.Cu") (net 3))
+  (segment (start 64.900489 54.825489) (end 62.05 51.975) (width 0.3) (layer "In1.Cu") (net 3))
+  (segment (start 58.7 49.25) (end 58.7 63.65) (width 0.3) (layer "In1.Cu") (net 3))
+  (segment (start 74.349511 56.449511) (end 63.8 45.9) (width 0.3) (layer "In1.Cu") (net 3))
+  (segment (start 74.349511 62.050489) (end 74.349511 56.449511) (width 0.3) (layer "In1.Cu") (net 3))
+  (segment (start 62.05 51.975) (end 62.05 50.675) (width 0.3) (layer "In1.Cu") (net 3))
+  (segment (start 63.8 45.9) (end 62.05 45.9) (width 0.3) (layer "In1.Cu") (net 3))
+  (segment (start 64.900489 68.500489) (end 64.900489 54.825489) (width 0.3) (layer "In1.Cu") (net 3))
+  (segment (start 72.75 61.375) (end 62.05 50.675) (width 0.3) (layer "In1.Cu") (net 3))
+  (segment (start 62.05 50.675) (end 62.05 45.9) (width 0.3) (layer "In1.Cu") (net 3))
+  (segment (start 62.05 45.9) (end 58.7 49.25) (width 0.3) (layer "In1.Cu") (net 3))
   (segment (start 66.5 56) (end 65.4 54.9) (width 0.5) (layer "In2.Cu") (net 3))
   (segment (start 65.29812 59.899511) (end 66.00188 59.899511) (width 0.5) (layer "In2.Cu") (net 3))
@@
   (segment (start 71.227728 52.948191) (end 71.321142 52.854777) (width 0.3) (layer "F.Cu") (net 5))
   (segment (start 68.866637 52.948191) (end 71.227728 52.948191) (width 0.3) (layer "F.Cu") (net 5))
+  (segment (start 58.8 32.45) (end 58.75 32.4) (width 0.3) (layer "F.Cu") (net 6))
+  (segment (start 58.8 34) (end 58.8 32.45) (width 0.3) (layer "F.Cu") (net 6))
   (segment (start 64.145 81.995) (end 64.145 84.195) (width 0.3) (layer "F.Cu") (net 6))
   (segment (start 63.4 81.25) (end 64.145 81.995) (width 0.3) (layer "F.Cu") (net 6))
@@
     (polygon
       (pts
-        (xy 80.8 27.3)
-        (xy 80.6 90)
-        (xy 50 90.05)
-        (xy 50 27.25)
+        (xy 79.67706 26.715699)
+        (xy 79.476116 89.996431)
+        (xy 51.55 90.050024)
+        (xy 51.550944 26.669292)
       )
     )
@@
     (polygon
       (pts
-        (xy 80.65 89.95)
-        (xy 50.05 90)
-        (xy 50.05 27.3)
-        (xy 80.7 27.3)
+        (xy 79.5501 89.949131)
+        (xy 51.55 90)
+        (xy 51.55 26.7)
+        (xy 79.6001 26.699131)
       )
     )
